File: hardware/vespa.kicad_sch (KiCad schematic)
At the start: 113 parts, among them Q1 Q_PMOS, SW1 SW_Push, SW10 SW_Push, SW11 SW_Push, SW12 SW_Push, SW13 SW_Push, SW14 SW_Push, SW15 SW_Push, SW16 SW_Push, SW17 SW_Push, SW18 SW_Push, SW19 SW_Push, SW2 SW_Push, SW20 SW_Push, SW21 SW_Push, SW22 SW_Push, SW23 SW_Push, SW24 SW_Push, SW25 SW_Push, SW26 SW_Push, SW27 SW_Push, SW28 SW_Push, SW29 SW_Push, SW3 SW_Push, SW30 SW_Push, SW31 SW_Push, SW32 SW_Push, SW33 SW_Push, SW34 SW_Push, SW35 SW_Push, SW36 SW_Push, SW37 SW_Push, SW38 SW_Push, SW39 SW_Push, SW4 SW_Push, SW40 SW_Push, SW41 SW_Push, SW42 SW_Push, SW43 SW_Push, SW44 SW_Push, SW45 SW_Push, SW46 SW_Push, SW47 SW_Push, SW48 SW_Push, SW49 SW_Push, SW5 SW_Push, SW50 SW_Push, SW51 SW_Push, SW52 SW_Push, SW53 SW_SPDT, SW6 SW_Push, SW7 SW_Push, SW8 SW_Push, SW9 SW_Push, U1 XIAO nRF52840 Plus, U2 XCL103D333CR-G, U3 BU4210G-TR

Commit message: basic routing
Parts:
- added SW53: RotaryEncoder, My_lib:re111f, symbol Device:RotaryEncoder_Switch
- BT1: footprint (none) -> Battery:BatteryHolder_Keystone_2460_1xAA
- C1, C2: footprint (none) -> Capacitor_SMD:C_0603_1608Metric_Pad1.08x0.95mm_HandSolder
- D1, D10, D11, D12, D13, D14, D15, D16, D17, D18, D19, D2, D20, D21, D22, D23, D24, D25, D26, D27, D28, D29, D3, D30, D31, D32, D33, D34, D35, D36, D37, D38, D39, D4, D40, D41, D42, D43, D44, D45, D46, D47, D48, D49, D5, D50, D51, D52, D6, D7, D8, D9: footprint (none) -> Diode_SMD:D_SOD-323_HandSoldering
- Q1: footprint (none) -> Package_TO_SOT_SMD:SOT-23-3; symbol Device:Q_PMOS -> Transistor_FET:Q_PMOS_GSD
- R1: footprint (none) -> Resistor_SMD:R_0603_1608Metric_Pad0.98x0.95mm_HandSolder
- SW1, SW10, SW11, SW12, SW13, SW14, SW15, SW16, SW17, SW18, SW19, SW2, SW20, SW21, SW22, SW23, SW24, SW25, SW26, SW27, SW28, SW29, SW3, SW30, SW31, SW32, SW33, SW34, SW35, SW36, SW37, SW38, SW39, SW4, SW40, SW41, SW42, SW43, SW44, SW45, SW46, SW47, SW48, SW49, SW5, SW50, SW51, SW52, SW6, SW7, SW8, SW9: footprint (none) -> kbd_SW_PCBA:MX_Choc_v1v2_Hotswap_1u
- SW54: renamed from SW53; footprint (none) -> My_lib:SS-12D00
- U1: footprint (none) -> My_lib:XIAO-nRF52840-Plus-SMD
- U2: footprint (none) -> My_lib:CL2025-02
- U3: footprint (none) -> My_lib:SSOP5
Connections:
- net +BATT: now also BT1.1 (+); no longer SW54.3 (C)
- net GND: now also SW54.3 (C), SW53.C; no longer BT1.2 (-)
- net VBUS: now also Q1.1 (G); no longer Q1.G
- net VCC: now also Q1.2 (S); no longer Q1.S
- net col1: now also U1.23 (D19/P1.07); no longer U1.10 (D9/1.14)
- net col10: now also U1.15 (D11/P0.15); no longer U1.5 (D4/0.04)
- net col11: now also U1.1 (D0/0.02); no longer U1.6 (D5/0.05)
- net col2: now also U1.10 (D9/1.14); no longer U1.9 (D8/1.13)
- net col3: now also U1.22 (D18/P1.05); no longer U1.8 (D7/1.12)
- net col4: now also U1.21 (D17/P1.03); no longer U1.23 (D19/P1.07)
- net col5: now also U1.9 (D8/1.13), SW53.S2; no longer U1.22 (D18/P1.05)
- net col6: now also U1.3 (D2/0.28); no longer U1.1 (D0/0.02)
- net col7: now also U1.4 (D3/0.29); no longer U1.2 (D1/0.03)
- net col8: now also U1.16 (D12/P0.19); no longer U1.3 (D2/0.28)
- net col9: now also U1.2 (D1/0.03); no longer U1.4 (D3/0.29)
- net row0: now also U1.17 (D13/P1.01); no longer U1.21 (D17/P1.03)
- net row1: now also U1.5 (D4/0.04); no longer U1.7 (D6/1.11)
- net row2: now also U1.6 (D5/0.05); no longer U1.15 (D11/P0.15)
- net row3: now also U1.7 (D6/1.11); no longer U1.16 (D12/P0.19)
- net row4: now also U1.8 (D7/1.12), SW53.S1; no longer U1.17 (D13/P1.01)
- net at C2.1, U2.6 (VOUT): now also Q1.3 (D); no longer Q1.D
- net reA: now reaches U1.18 (D14/P0.09)
- net reA: now also SW53.A
- net reB: now reaches U1.19 (D15/P0.10)
- net reB: now also SW53.B
- net at SW54.2 (B): now also BT1.2 (-); no longer BT1.1 (+)
- no-connect marks 7 -> 5
Other:
- moved on the sheet: SW54

Commit message: update pcb
Parts:
- SW54: footprint My_lib:SS-12D00 -> My_lib:SW_SPDT_IS-1245T
Connections:
- net GND: now also SW54.1 (A); no longer SW54.3 (C)
- net row2: now also U1.7 (D6/1.11); no longer U1.6 (D5/0.05)
- net row3: now also U1.6 (D5/0.05); no longer U1.7 (D6/1.11)
Changed lines of the file:
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@@
 	)
 	(no_connect
-		(at 44.45 139.7)
-	)
-	(no_connect
 		(at 54.61 76.2)
 	)
@@
 	)
 	(no_connect
+		(at 44.45 139.7)
+	)
+	(no_connect
 		(at 81.28 153.67)
 	)
@@
 	)
 	(label "row2"
-		(at 29.21 53.34 180)
+		(at 29.21 55.88 180)
 		(effects
 			(font
@@
 	)
 	(label "row3"
-		(at 29.21 55.88 180)
+		(at 29.21 53.34 180)
 		(effects
 			(font
@@
 		(lib_id "Switch:SW_SPDT")
 		(at 39.37 137.16 0)
-		(mirror x)
 		(unit 1)
 		(exclude_from_sim no)
@@
 		(dnp no)
 		(property "Reference" "SW54"
-			(at 39.37 146.05 0)
+			(at 39.37 128.27 0)
 			(effects
 				(font
@@
 		)
 		(property "Value" "SW_SPDT"
-			(at 39.37 143.51 0)
+			(at 39.37 130.81 0)
 			(effects
 				(font
@@
 			)
 		)
-		(property "Footprint" "My_lib:SS-12D00"
+		(property "Footprint" "My_lib:SW_SPDT_IS-1245T"
 			(at 39.37 137.16 0)
 			(effects
@@
 			)
 		)
-		(property "Datasheet" "~"
-			(at 39.37 129.54 0)
+		(property "Datasheet" "https://akizukidenshi.com/catalog/g/g115368/"
+			(at 39.37 144.78 0)
 			(effects
 				(font
