File: hardware/vespa.kicad_pcb (KiCad board)
At the start: 2 copper layers, 256.5 x 100.3 mm, 114 parts, among them Q1 Q_PMOS, SW1 SW_Push, SW10 SW_Push, SW11 SW_Push, SW12 SW_Push, SW13 SW_Push, SW14 SW_Push, SW15 SW_Push, SW16 SW_Push, SW17 SW_Push, SW18 SW_Push, SW19 SW_Push, SW2 SW_Push, SW20 SW_Push, SW21 SW_Push, SW22 SW_Push, SW23 SW_Push, SW24 SW_Push, SW25 SW_Push, SW26 SW_Push, SW27 SW_Push, SW28 SW_Push, SW29 SW_Push, SW3 SW_Push, SW30 SW_Push, SW31 SW_Push, SW32 SW_Push, SW33 SW_Push, SW34 SW_Push, SW35 SW_Push, SW36 SW_Push, SW37 SW_Push, SW38 SW_Push, SW39 SW_Push, SW4 SW_Push, SW40 SW_Push, SW41 SW_Push, SW42 SW_Push, SW43 SW_Push, SW44 SW_Push, SW45 SW_Push, SW46 SW_Push, SW47 SW_Push, SW48 SW_Push, SW49 SW_Push, SW5 SW_Push, SW50 SW_Push, SW51 SW_Push, SW52 SW_Push, SW53 RotaryEncoder, SW54 SW_SPDT, SW6 SW_Push, SW7 SW_Push, SW8 SW_Push, SW9 SW_Push, U1 XIAO nRF52840 Plus, U2 XCL103D333CR-G, U3 BU4210G-TR

Commit message: update pcb
Parts:
- added Ref**: Val**, kbd_Hole:m2_Spacer_Hole, F.Cu at (156.8, 88.9)
- added Ref**: Val**, kbd_Hole:m2_Spacer_Hole, F.Cu at (179.7, 88.9)
- added Ref**: Val**, kbd_Hole:m2_Spacer_Hole, F.Cu at (117.5, 145.4)
- added Ref**: Val**, kbd_Hole:m2_Spacer_Hole, F.Cu at (219.1, 145.4)
- SW54: footprint My_lib:SS-12D00 -> My_lib:SW_SPDT_IS-1245T
- moved SW54 0.44 mm to (168.3, 145.3), turned to 180 degrees
Connections:
- SW54 pad 1: unconnected-(SW54-A-Pad1) -> GND
- SW54 pad 3: GND -> unconnected-(SW54-C-Pad3)
- U1 pad 6: /row2 -> /row3
- U1 pad 7: /row3 -> /row2
Routing:
- net /col8: track 163.9 -> 185.9 mm
- net /col4: track 159.1 -> 181.1 mm
- net /row3: track 309.9 -> 313.2 mm
- net /row2: track 291.7 -> 288.6 mm
- net Net-(BT1--): track 5.08 -> 6.24 mm
- net /row4: track 210.6 -> 209.6 mm
- net /row1: track 275.9 -> 276.2 mm, vias 0 -> 1

Commit message: plate v1
Parts:
- removed the Ref** at (117.5, 145.4)
- removed the Ref** at (219.1, 145.4)
- added G***: LOGO, LOGO, B.Cu at (142.9, 149.2)
- added Ref**: Val**, kbd_Hole:m2_Spacer_Hole, F.Cu at (214.0, 145.4)
- added Ref**: Val**, kbd_Hole:m2_Spacer_Hole, F.Cu at (122.6, 145.4)
- AA Battery: renamed from BT1
Routing:
- net /col8: track 185.9 -> 163.9 mm
- net /col4: track 181.1 -> 159.1 mm
Other:
- outline, holes or cut-outs redrawn
- board text added: "Designed by object1037"
- board text added: "Vespa"

Commit message: update
Parts:
- moved G*** 2.54 mm to (142.9, 146.7)
Routing:
- net GND: track 28.1 -> 22.8 mm
- net /row4: track 209.6 -> 207.2 mm
- net /row1: vias 1 -> 0
