File: hardware/vespa_bottom_plate.kicad_pcb (KiCad board)
At the start: 2 copper layers, 273.1 x 100.3 mm, 8 parts

Commit message: update
Parts:
- added G***: LOGO, LOGO, B.Cu at (177.8, 68.6)
- moved Ref** 9.53 mm to (300.4, 138.4)
- moved Ref** 9.53 mm to (36.2, 138.4)
- moved Ref** 9.52 mm to (300.4, 71.1)
- moved Ref** 9.52 mm to (36.2, 71.1)
Other:
- outline, holes or cut-outs redrawn
