File: hardware/vespa_plate.kicad_pcb (KiCad board)
At the start: 2 copper layers, 273.1 x 100.3 mm, 60 parts, among them SW2 KEY_SWITCH

Commit message: update
Parts:
- moved Ref** 9.53 mm to (300.4, 138.4)
- moved Ref** 9.53 mm to (36.2, 138.4)
- moved Ref** 9.52 mm to (300.4, 71.1)
- moved Ref** 9.52 mm to (36.2, 71.1)
Other:
- outline, holes or cut-outs redrawn
Changed lines of the file:
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@@
 	(footprint "kbd_Hole:m2_Screw_Hole"
 		(layer "F.Cu")
-		(at 300.355 80.645)
+		(at 300.355 71.12)
 		(descr "Mounting Hole 2.2mm, no annular, M2")
 		(tags "mounting hole 2.2mm no annular m2")
@@
 	(footprint "kbd_Hole:m2_Screw_Hole"
 		(layer "F.Cu")
-		(at 36.195 80.645)
+		(at 36.195 71.12)
 		(descr "Mounting Hole 2.2mm, no annular, M2")
 		(tags "mounting hole 2.2mm no annular m2")
@@
 	(footprint "kbd_Hole:m2_Screw_Hole"
 		(layer "F.Cu")
-		(at 300.355 128.905)
+		(at 300.355 138.43)
 		(descr "Mounting Hole 2.2mm, no annular, M2")
 		(tags "mounting hole 2.2mm no annular m2")
@@
 	(footprint "kbd_Hole:m2_Screw_Hole"
 		(layer "F.Cu")
-		(at 36.195 128.905)
+		(at 36.195 138.43)
 		(descr "Mounting Hole 2.2mm, no annular, M2")
 		(tags "mounting hole 2.2mm no annular m2")
@@
 		(layer "Edge.Cuts")
 	)
+	(gr_arc
+		(start 36.195 142.875)
+		(mid 33.05191 141.57309)
+		(end 31.75 138.43)
+		(stroke
+			(width 0.05)
+			(type default)
+		)
+		(locked yes)
+		(layer "Edge.Cuts")
+	)
 	(gr_line
 		(start 159.385 85.725)
@@
 	)
 	(gr_line
-		(start 302.26 66.675)
-		(end 34.29 66.675)
+		(start 300.355 66.675)
+		(end 36.195 66.675)
 		(stroke
 			(width 0.05)
@@
 		(layer "Edge.Cuts")
 	)
-	(gr_arc
-		(start 34.29 142.875)
-		(mid 32.493949 142.131051)
-		(end 31.75 140.335)
+	(gr_line
+		(start 239.395 164.465)
+		(end 239.395 145.415)
 		(stroke
 			(width 0.05)
@@
 	)
 	(gr_line
-		(start 239.395 164.465)
-		(end 239.395 145.415)
+		(start 177.523611 90.252221)
+		(end 177.44139 90.087779)
 		(stroke
 			(width 0.05)
 			(type default)
 		)
-		(locked yes)
 		(layer "Edge.Cuts")
 	)
-	(gr_line
-		(start 177.523611 90.252221)
-		(end 177.44139 90.087779)
+	(gr_arc
+		(start 31.75 71.12)
+		(mid 33.05191 67.97691)
+		(end 36.195 66.675)
 		(stroke
 			(width 0.05)
 			(type default)
 		)
+		(locked yes)
 		(layer "Edge.Cuts")
 	)
@@
 	)
 	(gr_arc
+		(start 304.8 138.43)
+		(mid 303.49809 141.57309)
+		(end 300.355 142.875)
+		(stroke
+			(width 0.05)
+			(type default)
+		)
+		(locked yes)
+		(layer "Edge.Cuts")
+	)
+	(gr_arc
 		(start 201.077102 167.005)
 		(mid 200.105086 166.811655)
@@
 		(layer "Edge.Cuts")
 	)
-	(gr_arc
-		(start 304.8 140.335)
-		(mid 304.056051 142.131051)
-		(end 302.26 142.875)
+	(gr_line
+		(start 159.10861 90.087779)
+		(end 159.026389 90.252221)
 		(stroke
 			(width 0.05)
 			(type default)
 		)
-		(locked yes)
 		(layer "Edge.Cuts")
 	)
 	(gr_arc
-		(start 302.26 66.675)
-		(mid 304.056051 67.418949)
-		(end 304.8 69.215)
+		(start 300.355 66.675)
+		(mid 303.49809 67.97691)
+		(end 304.8 71.12)
 		(stroke
 			(width 0.05)
@@
 	)
 	(gr_line
-		(start 159.10861 90.087779)
-		(end 159.026389 90.252221)
-		(stroke
-			(width 0.05)
-			(type default)
-		)
-		(layer "Edge.Cuts")
-	)
-	(gr_line
-		(start 302.26 142.875)
+		(start 300.355 142.875)
 		(end 241.935 142.875)
 		(stroke
@@
 	)
 	(gr_line
-		(start 304.8 140.335)
-		(end 304.8 69.215)
+		(start 304.8 138.43)
+		(end 304.8 71.12)
 		(stroke
 			(width 0.05)
@@
 	)
 	(gr_arc
-		(start 31.75 69.215)
-		(mid 32.493949 67.418949)
-		(end 34.29 66.675)
-		(stroke
-			(width 0.05)
-			(type default)
-		)
-		(locked yes)
-		(layer "Edge.Cuts")
-	)
-	(gr_arc
 		(start 99.695 167.005)
 		(mid 97.898949 166.261051)
@@
 	)
 	(gr_line
-		(start 34.29 142.875)
+		(start 36.195 142.875)
 		(end 94.615 142.875)
 		(stroke
@@
 	)
 	(gr_line
-		(start 31.75 69.215)
-		(end 31.75 140.335)
+		(start 31.75 71.12)
+		(end 31.75 138.43)
 		(stroke
 			(width 0.05)
@@
 			)
 		)
+	)
+	(zone
+		(net 0)
+		(net_name "")
+		(layers "F.Cu" "B.Cu")
+		(name "Ant")
+		(hatch edge 0.5)
+		(connect_pads
+			(clearance 0)
+		)
+		(min_thickness 0.25)
+		(filled_areas_thickness no)
+		(keepout
+			(tracks allowed)
+			(vias allowed)
+			(pads allowed)
+			(copperpour not_allowed)
+			(footprints allowed)
+		)
+		(placement
+			(enabled no)
+			(sheetname "")
+		)
+		(fill
+			(thermal_gap 0.5)
+			(thermal_bridge_width 0.5)
+		)
+		(polygon
+			(pts
+				(xy 155.575 66.675) (xy 155.575 88.9) (xy 180.975 88.9) (xy 180.975 66.675)
+			)
+		)
